Commit message: add the lifting plarform controller into the ros2 control urdf config

File: cp15_auxiliary_files/rb1_ros2_description/urdf/common.gazebo.xacro (robot description, xacro)
@@ -23,7 +23,17 @@
                 <state_interface name="position" />
             </joint>
+            <joint name="robot_elevator_platform_joint">
+                <command_interface name="effort">
+                    <param name="min">0</param>
+                    <param name="max">10</param>
+                </command_interface>
+                <state_interface name="position"/>
+                <state_interface name="velocity"/>
+                <state_interface name="effort"/>
+            </joint>
         </ros2_control>
         <gazebo>
             <plugin filename="libgazebo_ros2_control.so" name="gazebo_ros2_control">
+                <robot_sim_type>gazebo_ros2_control/DefaultRobotHWSim</robot_sim_type>
                 <parameters>$(find rb1_ros2_description)/config/rb1_controller.yaml</parameters>
             </plugin>
